Commit message: katana_description: update katana_300_6m180.urdf.xacro
original author: Steffen Pfiffner <pfiffnst@hs-weingarten.de>

File: katana_description/urdf/katana_300_6m180.urdf.xacro (robot description, xacro)
@@ -14,4 +14,5 @@
   <property name="link4_length" value="0.1523" />
   <property name="link5_length" value="0.1505" />
+  <property name="tool_frame_offset" value="-0.19" />
   <!-- All inertial values (mass, center of mass and inertia tensor) have been
        calculated from the meshes using MeshLab -->
@@ -212,4 +213,25 @@
       </inertial>
     </link>
+    <joint name="katana_motor5_wrist_roll_discs_joint" type="fixed">
+      <parent link="katana_motor5_wrist_roll_link" />
+      <child link="katana_motor5_wrist_roll_discs" />
+      <origin rpy="0 ${M_PI/2} 0" xyz="0.0375 0 0"/>
+    </joint>
+    <link name="katana_motor5_wrist_roll_discs">
+      <visual>
+        <origin xyz="0 0 0" rpy="0 0 0" />
+        <geometry>
+          <cylinder length="0.025" radius="0.025" />
+        </geometry>
+        <material name="grey" />
+      </visual>
+      <collision>
+        <origin xyz="0 0 0" rpy="0 0 0" />
+        <geometry>
+          <cylinder length="0.025" radius="0.025" />
+        </geometry>
+      </collision>
+      <xacro:cylinder_inertial length="0.025" radius="0.025"  mass="0.05" />
+    </link>
     <joint name="katana_gripper_joint" type="fixed">
       <parent link="katana_motor5_wrist_roll_link" />
@@ -244,9 +266,9 @@
         <origin rpy="${rotate} 0 0" xyz="0.034 0 0"/>
         <axis xyz="0 0 1"/>
-        <limit effort="0.5" lower="-0.44" upper="0.30"  velocity="0.718834"/>
+        <limit effort="0.5" lower="-0.85" upper="0.30"  velocity="1"/>
       </joint>
       <link name="katana_${prefix}_finger_link">
         <visual>
-          <origin rpy="0 ${M_PI} 0" xyz="0 0 0"/>
+          <origin rpy="0 ${M_PI} 0.27" xyz="0 0 0"/>
           <geometry>
             <mesh filename="package://katana_description/meshes/katana/katana_gripper_${prefix}_finger.stl"/>
@@ -255,5 +277,5 @@
         </visual>
         <collision>
-          <origin rpy="0 ${M_PI} 0" xyz="0 0 0"/>
+          <origin rpy="0 ${M_PI} 0.27" xyz="0 0 0"/>
           <geometry>
             <mesh filename="package://katana_description/meshes/katana/convex/katana_gripper_${prefix}_finger_convex.stl"/>
@@ -274,5 +296,5 @@
       <parent link="katana_motor5_wrist_roll_link"/>
       <child link="katana_gripper_tool_frame" />
-      <origin xyz="0 0 -${link5_length}" rpy="0 ${M_PI/2} 0"/>
+      <origin xyz="0 0 ${tool_frame_offset}" rpy="0 ${M_PI/2} 0"/>
     </joint>
     <link name="katana_gripper_tool_frame">
